Commit message: meshes追加

File: urdf/body.urdf.xacro (robot description, xacro)
@@ -5,13 +5,15 @@
         <link name="base_link">
             <collision>
-                <origin xyz="0 0 0.45" rpy="0 0 0" />
+                <origin xyz="0 0 0.0" rpy="0 0 0" />
                 <geometry>
-                    <box size="0.5 0.33 0.7" />
+                    <!-- <box size="0.5 0.33 0.7" /> -->
+                    <mesh filename="file://$(find xarm_shuidi_description)/meshes/shuidi_agv.stl"/>
                 </geometry>
             </collision>
             <visual>
-                <origin xyz="0 0 0.45" rpy="0 0 0" />
+                <origin xyz="0 0 0.0" rpy="0 0 0" />
                 <geometry>
-                    <box size="0.5 0.33 0.7" />
+                    <!-- <box size="0.5 0.33 0.7" /> -->
+                     <mesh filename="file://$(find xarm_shuidi_description)/meshes/shuidi_agv.stl"/>
                 </geometry>
                 <material name="white">

File: urdf/caster.urdf.xacro (robot description, xacro)
@@ -1,22 +1,22 @@
 <?xml version="1.0"?>
 <robot xmlns:xacro="http://www.ros.org/wiki/xacro" name="caster">
-    <xacro:macro name="caster" params="parent xyz:='0 0 0' rpy:='0 0 0'">
-        <joint name="caster_joint" type="fixed">
+    <xacro:macro name="caster" params="prefix parent xyz:='0 0 0' rpy:='0 0 0'">
+        <joint name="${prefix}_caster_joint" type="fixed">
             <origin xyz="${xyz}" rpy="${rpy}" />
             <parent link="${parent}" />
-            <child link="caster" />
+            <child link="${prefix}_caster" />
         </joint>
-        <transmission name="caster_trans" type="SimpleTransmission">
+        <transmission name="${prefix}_caster_trans" type="SimpleTransmission">
             <type>transmission_interface/SimpleTransmission</type>
-            <actuator name="caster_motor">
+            <actuator name="${prefix}_caster_motor">
                 <!-- ギア比 -->
                 <mechanicalReduction>1</mechanicalReduction>
             </actuator>
-            <joint name="caster_joint">
+            <joint name="${prefix}_caster_joint">
                 <hardwareInterface>hardware_interface/VelocityJointInterface</hardwareInterface>
             </joint>
         </transmission>
         <!-- caster frontal wheel Link -->
-        <link name="caster">
+        <link name="${prefix}_caster">
             <collision>
                 <geometry>
@@ -44,5 +44,5 @@
             </inertial>
         </link>
-        <gazebo reference="caster">
+        <gazebo reference="${prefix}_caster">
             <material>Gazebo/Blue</material>
             <!-- 摩擦係数はとりあえず0にして引っかからないようにする -->

File: urdf/shuidi.urdf.xacro (robot description, xacro)
@@ -8,9 +8,10 @@
     <xacro:include filename="$(find xarm_shuidi_description)/xacro/imu.xacro" />
     <xacro:body />
-    <xacro:wheel prefix="left" parent="base_link" xyz="0.125 0.21 0.125" rpy="-1.5707 0 0" />
-    <xacro:wheel prefix="right" parent="base_link" xyz="0.125 -0.21 0.125" rpy="-1.5707 0 0" />
-    <xacro:caster parent="base_link" xyz="-0.25 0 0.05" rpy="1.57 0 0" />
-    <xacro:lidar parent="base_link" xyz="0.3 0 0.28" rpy="0 0 0" />
-    <xacro:imu parent="base_link" xyz="0 0 0.8" rpy="0 0 0" />
+    <xacro:wheel prefix="left" parent="base_link" xyz="0 0.18 0.059" rpy="-1.5707 0 0" />
+    <xacro:wheel prefix="right" parent="base_link" xyz="0 -0.18 0.059" rpy="-1.5707 0 0" />
+    <xacro:caster prefix="front" parent="base_link" xyz="0.097 0 0.034" rpy="1.57 0 0" />
+    <xacro:caster prefix="rear" parent="base_link" xyz="-0.14 0 0.034" rpy="1.57 0 0" />
+    <!-- <xacro:lidar parent="base_link" xyz="0.3 0 0.28" rpy="0 0 0" />
+    <xacro:imu parent="base_link" xyz="0 0 0.8" rpy="0 0 0" /> -->
     <xacro:diff_drive_control left_joint="left_wheel_joint" right_joint="right_wheel_joint" />
     <gazebo>

File: urdf/wheel.urdf.xacro (robot description, xacro)
@@ -24,10 +24,10 @@
             <collision>
                 <geometry>
-                    <cylinder radius="0.125" length="0.085" />
+                    <cylinder radius="0.075" length="0.045" />
                 </geometry>
             </collision>
             <visual>
                 <geometry>
-                    <cylinder radius="0.125" length="0.085" />
+                    <cylinder radius="0.075" length="0.045" />
                 </geometry>
                 <material name="red">

Commit message: ファイル構造をturtlebotに準拠

File: urdf/body.urdf.xacro (robot description, xacro)
@@ -33,7 +33,4 @@
             </inertial>
         </link>
-        <gazebo reference="base_link">
-            <material>Gazebo/White</material>
-        </gazebo>
     </xacro:macro>
 </robot>

File: urdf/caster.urdf.xacro (robot description, xacro)
@@ -44,10 +44,4 @@
             </inertial>
         </link>
-        <gazebo reference="${prefix}_caster">
-            <material>Gazebo/Blue</material>
-            <!-- 摩擦係数はとりあえず0にして引っかからないようにする -->
-            <mu1>0.0</mu1>
-            <mu2>0.0</mu2>
-        </gazebo>
     </xacro:macro>
 </robot>

File: urdf/shuidi.urdf.xacro (robot description, xacro)
@@ -1,47 +1,18 @@
 <?xml version="1.0"?>
-<robot name="diff_drive" xmlns:xacro="http://www.ros.org/wiki/xacro">
-    <xacro:include filename="$(find xarm_shuidi_description)/urdf/wheel.urdf.xacro" />
-    <xacro:include filename="$(find xarm_shuidi_description)/ros2_control/shuidi.ros2_control.xacro" />
-    <xacro:include filename="$(find xarm_shuidi_description)/urdf/body.urdf.xacro" />
-    <xacro:include filename="$(find xarm_shuidi_description)/urdf/caster.urdf.xacro" />
-    <xacro:include filename="$(find xarm_shuidi_description)/xacro/lidar.xacro" />
-    <xacro:include filename="$(find xarm_shuidi_description)/xacro/imu.xacro" />
-    <xacro:body />
-    <xacro:wheel prefix="left" parent="base_link" xyz="0 0.18 0.059" rpy="-1.5707 0 0" />
-    <xacro:wheel prefix="right" parent="base_link" xyz="0 -0.18 0.059" rpy="-1.5707 0 0" />
-    <xacro:caster prefix="front" parent="base_link" xyz="0.097 0 0.034" rpy="1.57 0 0" />
-    <xacro:caster prefix="rear" parent="base_link" xyz="-0.14 0 0.034" rpy="1.57 0 0" />
-    <!-- <xacro:lidar parent="base_link" xyz="0.3 0 0.28" rpy="0 0 0" />
-    <xacro:imu parent="base_link" xyz="0 0 0.8" rpy="0 0 0" /> -->
-    <xacro:diff_drive_control left_joint="left_wheel_joint" right_joint="right_wheel_joint" />
-    <gazebo>
-        <!-- Joint state publisher -->
-        <plugin filename="libgazebo_ros2_control.so" name="gazebo_ros2_control">
-            <robot_param>robot_description</robot_param>
-            <robot_param_node>robot_state_publisher</robot_param_node>
-            <parameters>$(find xarm_shuidi_description)/config/diff_drive_controller.yaml</parameters>
-        </plugin>
-        <!-- <plugin name="diff_drive" filename="libgazebo_ros_diff_drive.so">
-            <ros>
-                <remapping>cmd_vel:=cmd_vel</remapping>
-                <namespace>/diff_drive_base_controller</namespace>
-                <remapping>odom:=odom</remapping>
-            </ros>
-            <left_joint>left_wheel_joint</left_joint>
-            <right_joint>right_wheel_joint</right_joint>
-            <wheel_separation>0.42</wheel_separation>
-            <wheel_radius>0.125</wheel_radius>
-            <max_wheel_torque>20</max_wheel_torque>
-            <max_wheel_acceleration>1.0</max_wheel_acceleration>
-            <publish_odom>true</publish_odom>
-            <publish_odom_tf>false</publish_odom_tf>
-            <publish_wheel_tf>true</publish_wheel_tf>
-            <update_rate>30</update_rate>
-            <odometry_topic>odom</odometry_topic>
-            <odometry_frame>odom</odometry_frame>
-            <base_frame_id>base_link</base_frame_id>
-            <robot_base_frame>base_link</robot_base_frame>
-            <command_topic>cmd_vel</command_topic>
-        </plugin> -->
-    </gazebo>
+<robot  xmlns:xacro="http://www.ros.org/wiki/xacro">
+    <xacro:macro name="shuidi">
+        <xacro:include filename="$(find xarm_shuidi_description)/urdf/wheel.urdf.xacro" />
+        <xacro:include filename="$(find xarm_shuidi_description)/urdf/body.urdf.xacro" />
+        <xacro:include filename="$(find xarm_shuidi_description)/urdf/caster.urdf.xacro" />
+        <xacro:include filename="$(find xarm_shuidi_description)/xacro/lidar.xacro" />
+        <xacro:include filename="$(find xarm_shuidi_description)/xacro/imu.xacro" />
+        <xacro:body />
+        <xacro:wheel prefix="left" parent="base_link" xyz="0 0.18 0.059" rpy="-1.5707 0 0" />
+        <xacro:wheel prefix="right" parent="base_link" xyz="0 -0.18 0.059" rpy="-1.5707 0 0" />
+        <xacro:caster prefix="front" parent="base_link" xyz="0.097 0 0.034" rpy="1.57 0 0" />
+        <xacro:caster prefix="rear" parent="base_link" xyz="-0.14 0 0.034" rpy="1.57 0 0" />
+        <!-- sensor -->
+        <!-- <xacro:lidar parent="base_link" xyz="0.3 0 0.28" rpy="0 0 0" />
+        <xacro:imu parent="base_link" xyz="0 0 0.8" rpy="0 0 0" /> -->
+    </xacro:macro>
 </robot>

File: urdf/wheel.urdf.xacro (robot description, xacro)
@@ -45,7 +45,4 @@
             </inertial>
         </link>
-        <gazebo reference="${prefix}_wheel">
-            <material>Gazebo/Red</material>
-        </gazebo>
     </xacro:macro>
 </robot>
