Commit message: make xarm_shuidi urdf file

File: gazebo/shuidi.gazebo.xacro (robot description, xacro)
@@ -1,15 +1,18 @@
 <?xml version="1.0"?>
 <robot xmlns:xacro="http://www.ros.org/wiki/xacro">
-    <xacro:macro name="shuidi_gazebo">
-        <gazebo reference="left_wheel">
+    <xacro:macro name="shuidi_gazebo" params="prefix">
+        <gazebo reference="${prefix}left_wheel">
                 <material>Gazebo/Red</material>
         </gazebo>
-        <gazebo reference="right_wheel">
+        <gazebo reference="${prefix}right_wheel">
                 <material>Gazebo/Red</material>
         </gazebo>
-        <gazebo reference="base_link">
+        <gazebo reference="${prefix}base_link">
             <material>Gazebo/White</material>
         </gazebo>
-        <gazebo reference="front_caster">
+        <gazebo reference="${prefix}battery">
+            <material>Gazebo/White</material>
+        </gazebo>
+        <gazebo reference="${prefix}front_caster">
             <material>Gazebo/Blue</material>
             <!-- 摩擦係数はとりあえず0にして引っかからないようにする -->
@@ -17,5 +20,5 @@
             <mu2>0.0</mu2>
         </gazebo>
-        <gazebo reference="rear_caster">
+        <gazebo reference="${prefix}rear_caster">
             <material>Gazebo/Blue</material>
             <!-- 摩擦係数はとりあえず0にして引っかからないようにする -->

File: urdf/components/body.urdf.xacro (robot description, xacro)
@@ -1,7 +1,7 @@
 <?xml version="1.0"?>
 <robot xmlns:xacro="http://www.ros.org/wiki/xacro" name="body">
-    <xacro:macro name="body" params="">
+    <xacro:macro name="body" params="prefix">
         <!-- Base Link -->
-        <link name="base_link">
+        <link name="${prefix}base_link">
             <collision>
                 <origin xyz="0 0 0.0" rpy="0 0 0" />

File: urdf/shuidi.urdf.xacro (robot description, xacro)
@@ -1,15 +1,17 @@
 <?xml version="1.0"?>
 <robot  xmlns:xacro="http://www.ros.org/wiki/xacro">
-    <xacro:macro name="shuidi">
+    <xacro:macro name="shuidi" params="prefix">
         <xacro:include filename="$(find xarm_shuidi_description)/urdf/components/wheel.urdf.xacro" />
         <xacro:include filename="$(find xarm_shuidi_description)/urdf/components/body.urdf.xacro" />
         <xacro:include filename="$(find xarm_shuidi_description)/urdf/components/caster.urdf.xacro" />
+        <xacro:include filename="$(find xarm_shuidi_description)/urdf/components/batteries.urdf.xacro" />
         <xacro:include filename="$(find xarm_shuidi_description)/gazebo/lidar.xacro" />
         <xacro:include filename="$(find xarm_shuidi_description)/gazebo/imu.xacro" />
-        <xacro:body />
-        <xacro:wheel prefix="left" parent="base_link" xyz="0 0.18 0.059" rpy="-1.5707 0 0" />
-        <xacro:wheel prefix="right" parent="base_link" xyz="0 -0.18 0.059" rpy="-1.5707 0 0" />
-        <xacro:caster prefix="front" parent="base_link" xyz="0.097 0 0.034" rpy="1.57 0 0" />
-        <xacro:caster prefix="rear" parent="base_link" xyz="-0.14 0 0.034" rpy="1.57 0 0" />
+        <xacro:body prefix="${prefix}"/>
+        <xacro:wheel prefix="${prefix}left" parent="${prefix}base_link" xyz="0 0.18 0.059" rpy="-1.5707 0 0" />
+        <xacro:wheel prefix="${prefix}right" parent="${prefix}base_link" xyz="0 -0.18 0.059" rpy="-1.5707 0 0" />
+        <xacro:caster prefix="${prefix}front" parent="${prefix}base_link" xyz="0.097 0 0.034" rpy="1.57 0 0" />
+        <xacro:caster prefix="${prefix}rear" parent="${prefix}base_link" xyz="-0.14 0 0.034" rpy="1.57 0 0" />
+        <xacro:battery prefix="${prefix}" parent="${prefix}base_link" xyz="0 0 0.277" rpy="0 0 0" />
         <!-- sensor -->
         <!-- <xacro:lidar parent="base_link" xyz="0.3 0 0.28" rpy="0 0 0" />

File: urdf/xarm_shuidi.urdf.xacro (robot description, xacro)
@@ -1,4 +1,7 @@
 <?xml version="1.0"?>
 <robot name="xarm_shuidi" xmlns:xacro="http://www.ros.org/wiki/xacro">
+    <!-- ここのprefixで全体にprefixがつく -->
+    <xacro:arg name="prefix" default=""/>
+    <!-- shuidi -->
     <!-- urdf -->
     <xacro:include filename="$(find xarm_shuidi_description)/urdf/shuidi.urdf.xacro" />
@@ -7,6 +10,62 @@
     <!-- ros2_control -->
     <xacro:include filename="$(find xarm_shuidi_description)/ros2_control/shuidi.ros2_control.xacro" />
-    <xacro:shuidi />
-    <xacro:shuidi_gazebo />
-    <xacro:diff_drive_control left_joint="left_wheel_joint" right_joint="right_wheel_joint" />
+    <xacro:shuidi prefix="$(arg prefix)"/>
+    <xacro:shuidi_gazebo prefix="$(arg prefix)"/>
+    <xacro:diff_drive_control left_joint="$(arg prefix)left_wheel_joint" right_joint="$(arg prefix)right_wheel_joint" />
+    <!-- xarm7 -->
+    <xacro:arg name="hw_ns" default="xarm"/>
+    <xacro:arg name="limited" default="false"/>
+    <xacro:arg name="effort_control" default="false"/>
+    <xacro:arg name="velocity_control" default="false"/>
+    <xacro:arg name="add_gripper" default="true"/>
+    <xacro:arg name="add_vacuum_gripper" default="false"/>
+    <xacro:arg name="model1300" default="false"/>
+    <xacro:arg name="dof" default="7"/>
+    <xacro:arg name="robot_ip" default=""/>
+    <xacro:arg name="robot_type" default="xarm"/>
+    <xacro:arg name="robot_sn" default=""/>
+    <xacro:arg name="report_type" default="normal"/>
+    <xacro:arg name="ros2_control_plugin" default="uf_robot_hardware/UFRobotSystemHardware"/>
+    <xacro:arg name="ros2_control_params" default=""/>
+    <xacro:arg name="add_realsense_d435i" default="false"/>
+    <xacro:arg name="add_d435i_links" default="true"/>
+    <xacro:arg name="use_gazebo_camera" default="false"/>
+    <xacro:arg name="add_other_geometry" default="false"/>
+    <xacro:arg name="geometry_type" default="box"/>
+    <xacro:arg name="geometry_mass" default="0.1"/>
+    <xacro:arg name="geometry_height" default="0.1"/>
+    <xacro:arg name="geometry_radius" default="0.1"/>
+    <xacro:arg name="geometry_length" default="0.1"/>
+    <xacro:arg name="geometry_width" default="0.1"/>
+    <xacro:arg name="geometry_mesh_filename" default=""/>
+    <xacro:arg name="geometry_mesh_origin_xyz" default="0 0 0"/>
+    <xacro:arg name="geometry_mesh_origin_rpy" default="0 0 0"/>
+    <xacro:arg name="geometry_mesh_tcp_xyz" default="0 0 0"/>
+    <xacro:arg name="geometry_mesh_tcp_rpy" default="0 0 0"/>
+    <xacro:arg name="baud_checkset" default="true"/>
+    <xacro:arg name="default_gripper_baud" default="2000000"/>
+    <xacro:arg name="attach_to" default="$(arg prefix)base_link"/>
+    <xacro:arg name="attach_xyz" default="0 0 0.446"/>
+    <xacro:arg name="attach_rpy" default="0 0 0"/>
+    <xacro:arg name="mesh_suffix" default="stl"/>
+    <xacro:arg name="kinematics_suffix" default=""/>
+    <xacro:include filename="$(find xarm_description)/urdf/xarm_device_macro.xacro" />
+    <xacro:xarm_device prefix="$(arg prefix)" hw_ns="$(arg hw_ns)" limited="$(arg limited)"
+    effort_control="$(arg effort_control)" velocity_control="$(arg velocity_control)"
+    add_gripper="$(arg add_gripper)" add_vacuum_gripper="$(arg add_vacuum_gripper)" dof="$(arg dof)"
+    ros2_control_plugin="$(arg ros2_control_plugin)" robot_type="$(arg robot_type)"
+    load_gazebo_plugin="true" ros2_control_params="$(arg ros2_control_params)"
+    add_realsense_d435i="$(arg add_realsense_d435i)"
+    add_d435i_links="$(arg add_d435i_links)"
+    add_other_geometry="$(arg add_other_geometry)"
+    geometry_type="$(arg geometry_type)" geometry_mass="$(arg geometry_mass)"
+    geometry_height="$(arg geometry_height)" geometry_radius="$(arg geometry_radius)"
+    geometry_length="$(arg geometry_length)" geometry_width="$(arg geometry_width)"
+    geometry_mesh_filename="$(arg geometry_mesh_filename)"
+    geometry_mesh_origin_xyz="$(arg geometry_mesh_origin_xyz)" geometry_mesh_origin_rpy="$(arg geometry_mesh_origin_rpy)"
+    geometry_mesh_tcp_xyz="$(arg geometry_mesh_tcp_xyz)" geometry_mesh_tcp_rpy="$(arg geometry_mesh_tcp_rpy)"
+    robot_ip="$(arg robot_ip)" report_type="$(arg report_type)"
+    baud_checkset="$(arg baud_checkset)" default_gripper_baud="$(arg default_gripper_baud)"
+    model1300="$(arg model1300)" attach_to="$(arg attach_to)" attach_xyz="$(arg attach_xyz)" attach_rpy="$(arg attach_rpy)"
+    robot_sn="$(arg robot_sn)" use_gazebo_camera="$(arg use_gazebo_camera)" mesh_suffix="$(arg mesh_suffix)" kinematics_suffix="$(arg kinematics_suffix)" />
 </robot>
