Commit message: あ

File: gazebo/shuidi.gazebo.xacro (robot description, xacro)
@@ -3,8 +3,12 @@
     <xacro:macro name="shuidi_gazebo" params="prefix">
         <gazebo reference="${prefix}left_wheel">
-                <material>Gazebo/Red</material>
+            <material>Gazebo/Red</material>
+            <mu1 value="0.5" />
+            <mu2 value="0.5" />
         </gazebo>
         <gazebo reference="${prefix}right_wheel">
-                <material>Gazebo/Red</material>
+            <material>Gazebo/Red</material>
+            <mu1 value="0.5" />
+            <mu2 value="0.5" />
         </gazebo>
         <gazebo reference="${prefix}base_link">
@@ -28,21 +32,22 @@
         <gazebo>
             <!-- Joint state publisher -->
-            <plugin filename="libgazebo_ros2_control.so" name="gazebo_ros2_control">
+            <!-- <plugin filename="libgazebo_ros2_control.so" name="gazebo_ros2_control">
                 <robot_param>robot_description</robot_param>
                 <robot_param_node>robot_state_publisher</robot_param_node>
-                <parameters>$(find xarm_shuidi_description)/config/diff_drive_controller.yaml</parameters>
-            </plugin>
-            <!-- <plugin name="diff_drive" filename="libgazebo_ros_diff_drive.so">
+                <parameters>$(find xarm_shuidi_bringup)/config/diff_drive_controller.yaml</parameters>
+            </plugin> -->
+            <plugin name="diff_drive" filename="libgazebo_ros_diff_drive.so">
                 <ros>
                     <remapping>cmd_vel:=cmd_vel</remapping>
-                    <namespace>/diff_drive_base_controller</namespace>
+                    <namespace>/diff_drive_${prefix}</namespace>
                     <remapping>odom:=odom</remapping>
                 </ros>
-                <left_joint>left_wheel_joint</left_joint>
-                <right_joint>right_wheel_joint</right_joint>
-                <wheel_separation>0.42</wheel_separation>
-                <wheel_radius>0.125</wheel_radius>
-                <max_wheel_torque>20</max_wheel_torque>
-                <max_wheel_acceleration>1.0</max_wheel_acceleration>
+                <left_joint>${prefix}left_wheel_joint</left_joint>
+                <right_joint>${prefix}right_wheel_joint</right_joint>
+                <wheel_separation>0.6</wheel_separation>
+                <!-- <wheel_radius>0.125</wheel_radius> -->
+                <wheel_diameter>0.2</wheel_diameter>
+                <max_wheel_torque>30</max_wheel_torque>
+                <max_wheel_acceleration>3.0</max_wheel_acceleration>
                 <publish_odom>true</publish_odom>
                 <publish_odom_tf>false</publish_odom_tf>
@@ -54,5 +59,5 @@
                 <robot_base_frame>base_link</robot_base_frame>
                 <command_topic>cmd_vel</command_topic>
-            </plugin> -->
+            </plugin>
         </gazebo>
     </xacro:macro>

File: urdf/components/batteries.urdf.xacro (robot description, xacro)
@@ -10,15 +10,24 @@
             <collision>
                 <geometry>
-                       <mesh filename="file://$(find xarm_shuidi_description)/meshes/battery.stl"/>
+                    <mesh filename="file://$(find xarm_shuidi_description)/meshes/battery.stl" />
                 </geometry>
             </collision>
             <visual>
                 <geometry>
-                       <mesh filename="file://$(find xarm_shuidi_description)/meshes/battery.stl"/>
+                    <mesh filename="file://$(find xarm_shuidi_description)/meshes/battery.stl" />
                 </geometry>
-               <material name="white">
+                <material name="white">
                     <color rgba="1 1 1 1" />
                 </material>
             </visual>
+            <inertial>
+                <mass value="5.0" />
+                <inertia ixx="0.3"
+                    ixy="0.0"
+                    ixz="0.0"
+                    iyy="0.3"
+                    iyz="0.0"
+                    izz="0.3" />
+            </inertial>
         </link>
         <joint name="${prefix}battery_fixture_joint" type="fixed">
@@ -30,10 +39,12 @@
             <collision>
                 <geometry>
-                       <mesh filename="file://$(find xarm_shuidi_description)/meshes/battery_fixture.stl"/>
+                    <mesh
+                        filename="file://$(find xarm_shuidi_description)/meshes/battery_fixture.stl" />
                 </geometry>
             </collision>
             <visual>
                 <geometry>
-                       <mesh filename="file://$(find xarm_shuidi_description)/meshes/battery_fixture.stl"/>
+                    <mesh
+                        filename="file://$(find xarm_shuidi_description)/meshes/battery_fixture.stl" />
                 </geometry>
                 <material name="white">

File: urdf/components/body.urdf.xacro (robot description, xacro)
@@ -8,5 +8,5 @@
                 <geometry>
                     <!-- <box size="0.5 0.33 0.7" /> -->
-                    <mesh filename="file://$(find xarm_shuidi_description)/meshes/shuidi_agv.stl"/>
+                    <mesh filename="file://$(find xarm_shuidi_description)/meshes/shuidi_agv.stl" />
                 </geometry>
             </collision>
@@ -15,5 +15,5 @@
                 <geometry>
                     <!-- <box size="0.5 0.33 0.7" /> -->
-                     <mesh filename="file://$(find xarm_shuidi_description)/meshes/shuidi_agv.stl"/>
+                    <mesh filename="file://$(find xarm_shuidi_description)/meshes/shuidi_agv.stl" />
                 </geometry>
                 <material name="white">
@@ -22,13 +22,13 @@
             </visual>
             <inertial>
-                <origin xyz="0 0 0.45" rpy="0 0 0" />
+                <origin xyz="0 0 0.2" rpy="0 0 0" />
                 <mass value="30" />
                 <inertia
-                    ixx="0.6"
+                    ixx="1.0"
                     ixy="0.0"
                     ixz="0.0"
-                    iyy="0.6"
+                    iyy="1.0"
                     iyz="0.0"
-                    izz="0.6" />
+                    izz="1.9" />
             </inertial>
         </link>

File: urdf/components/caster.urdf.xacro (robot description, xacro)
@@ -33,5 +33,5 @@
             </visual>
             <inertial>
-                <origin xyz="-0.957138 -0 0.2" rpy="0 0 0" />
+                <!-- <origin xyz="-0.957138 -0 0.2" rpy="0 0 0" /> -->
                 <mass value="1.1" />
                 <inertia

File: urdf/components/wheel.urdf.xacro (robot description, xacro)
@@ -24,10 +24,10 @@
             <collision>
                 <geometry>
-                    <cylinder radius="0.075" length="0.045" />
+                    <cylinder radius="0.1" length="0.045" />
                 </geometry>
             </collision>
             <visual>
                 <geometry>
-                    <cylinder radius="0.075" length="0.045" />
+                    <cylinder radius="0.1" length="0.045" />
                 </geometry>
                 <material name="red">

File: urdf/shuidi.urdf.xacro (robot description, xacro)
@@ -1,16 +1,22 @@
 <?xml version="1.0"?>
-<robot  xmlns:xacro="http://www.ros.org/wiki/xacro">
+<robot xmlns:xacro="http://www.ros.org/wiki/xacro">
     <xacro:macro name="shuidi" params="prefix">
         <xacro:include filename="$(find xarm_shuidi_description)/urdf/components/wheel.urdf.xacro" />
         <xacro:include filename="$(find xarm_shuidi_description)/urdf/components/body.urdf.xacro" />
         <xacro:include filename="$(find xarm_shuidi_description)/urdf/components/caster.urdf.xacro" />
-        <xacro:include filename="$(find xarm_shuidi_description)/urdf/components/batteries.urdf.xacro" />
+        <xacro:include
+            filename="$(find xarm_shuidi_description)/urdf/components/batteries.urdf.xacro" />
         <xacro:include filename="$(find xarm_shuidi_description)/gazebo/lidar.xacro" />
         <xacro:include filename="$(find xarm_shuidi_description)/gazebo/imu.xacro" />
-        <xacro:body prefix="${prefix}"/>
-        <xacro:wheel prefix="${prefix}left" parent="${prefix}base_link" xyz="0 0.18 0.059" rpy="-1.5707 0 0" />
-        <xacro:wheel prefix="${prefix}right" parent="${prefix}base_link" xyz="0 -0.18 0.059" rpy="-1.5707 0 0" />
-        <xacro:caster prefix="${prefix}front" parent="${prefix}base_link" xyz="0.097 0 0.034" rpy="1.57 0 0" />
-        <xacro:caster prefix="${prefix}rear" parent="${prefix}base_link" xyz="-0.14 0 0.034" rpy="1.57 0 0" />
+        <xacro:body prefix="${prefix}" />
+        <xacro:wheel prefix="${prefix}left" parent="${prefix}base_link" xyz="0 0.3 0.09"
+            rpy="-1.5707 0 0" />
+        <xacro:wheel prefix="${prefix}right" parent="${prefix}base_link" xyz="0 -0.3 0.09"
+            rpy="-1.5707 0 0" />
+        <xacro:caster prefix="${prefix}front" parent="${prefix}base_link" xyz="0.2 0 0.04"
+            rpy="1.57 0 0" />
+        <xacro:caster prefix="${prefix}rear" parent="${prefix}base_link" xyz="-0.2 0 0.04"
+            rpy="1.57 0 0"
+        />
         <xacro:battery prefix="${prefix}" parent="${prefix}base_link" xyz="0 0 0.277" rpy="0 0 0" />
         <!-- sensor -->

File: urdf/xarm_shuidi.urdf.xacro (robot description, xacro)
@@ -2,5 +2,5 @@
 <robot name="xarm_shuidi" xmlns:xacro="http://www.ros.org/wiki/xacro">
     <!-- ここのprefixで全体にprefixがつく -->
-    <xacro:arg name="prefix" default=""/>
+    <xacro:arg name="prefix" default="" />
     <!-- shuidi -->
     <!-- urdf -->
@@ -9,63 +9,72 @@
     <xacro:include filename="$(find xarm_shuidi_description)/gazebo/shuidi.gazebo.xacro" />
     <!-- ros2_control -->
-    <xacro:include filename="$(find xarm_shuidi_description)/ros2_control/shuidi.ros2_control.xacro" />
-    <xacro:shuidi prefix="$(arg prefix)"/>
-    <xacro:shuidi_gazebo prefix="$(arg prefix)"/>
-    <xacro:diff_drive_control left_joint="$(arg prefix)left_wheel_joint" right_joint="$(arg prefix)right_wheel_joint" />
+    <xacro:include
+        filename="$(find
+    xarm_shuidi_description)/ros2_control/shuidi.ros2_control.xacro" />
+    <xacro:shuidi prefix="$(arg prefix)" />
+    <xacro:shuidi_gazebo prefix="$(arg prefix)" />
+    <xacro:diff_drive_control left_joint="$(arg prefix)left_wheel_joint"
+        right_joint="$(arg prefix)right_wheel_joint" />
     <!-- xarm7 -->
-    <xacro:arg name="hw_ns" default="xarm"/>
-    <xacro:arg name="limited" default="false"/>
-    <xacro:arg name="effort_control" default="false"/>
-    <xacro:arg name="velocity_control" default="false"/>
-    <xacro:arg name="add_gripper" default="true"/>
-    <xacro:arg name="add_vacuum_gripper" default="false"/>
-    <xacro:arg name="model1300" default="false"/>
-    <xacro:arg name="dof" default="7"/>
-    <xacro:arg name="robot_ip" default=""/>
-    <xacro:arg name="robot_type" default="xarm"/>
-    <xacro:arg name="robot_sn" default=""/>
-    <xacro:arg name="report_type" default="normal"/>
-    <xacro:arg name="ros2_control_plugin" default="uf_robot_hardware/UFRobotSystemHardware"/>
-    <xacro:arg name="ros2_control_params" default=""/>
-    <xacro:arg name="add_realsense_d435i" default="false"/>
-    <xacro:arg name="add_d435i_links" default="true"/>
-    <xacro:arg name="use_gazebo_camera" default="false"/>
-    <xacro:arg name="add_other_geometry" default="false"/>
-    <xacro:arg name="geometry_type" default="box"/>
-    <xacro:arg name="geometry_mass" default="0.1"/>
-    <xacro:arg name="geometry_height" default="0.1"/>
-    <xacro:arg name="geometry_radius" default="0.1"/>
-    <xacro:arg name="geometry_length" default="0.1"/>
-    <xacro:arg name="geometry_width" default="0.1"/>
-    <xacro:arg name="geometry_mesh_filename" default=""/>
-    <xacro:arg name="geometry_mesh_origin_xyz" default="0 0 0"/>
-    <xacro:arg name="geometry_mesh_origin_rpy" default="0 0 0"/>
-    <xacro:arg name="geometry_mesh_tcp_xyz" default="0 0 0"/>
-    <xacro:arg name="geometry_mesh_tcp_rpy" default="0 0 0"/>
-    <xacro:arg name="baud_checkset" default="true"/>
-    <xacro:arg name="default_gripper_baud" default="2000000"/>
-    <xacro:arg name="attach_to" default="$(arg prefix)base_link"/>
-    <xacro:arg name="attach_xyz" default="0 0 0.446"/>
-    <xacro:arg name="attach_rpy" default="0 0 0"/>
-    <xacro:arg name="mesh_suffix" default="stl"/>
-    <xacro:arg name="kinematics_suffix" default=""/>
+    <xacro:arg name="hw_ns" default="xarm" />
+    <xacro:arg name="limited" default="false" />
+    <xacro:arg name="effort_control" default="false" />
+    <xacro:arg name="velocity_control" default="false" />
+    <xacro:arg name="add_gripper" default="true" />
+    <xacro:arg name="add_vacuum_gripper" default="false" />
+    <xacro:arg name="model1300" default="false" />
+    <xacro:arg name="dof" default="7" />
+    <xacro:arg name="robot_ip" default="" />
+    <xacro:arg name="robot_type" default="xarm" />
+    <xacro:arg name="robot_sn" default="" />
+    <xacro:arg name="report_type" default="normal" />
+    <xacro:arg name="ros2_control_plugin" default="uf_robot_hardware/UFRobotSystemHardware" />
+    <xacro:arg name="ros2_control_params" default="" />
+    <xacro:arg name="add_realsense_d435i" default="false" />
+    <xacro:arg name="add_d435i_links" default="true" />
+    <xacro:arg name="use_gazebo_camera" default="false" />
+    <xacro:arg name="add_other_geometry" default="false" />
+    <xacro:arg name="geometry_type" default="box" />
+    <xacro:arg name="geometry_mass" default="0.1" />
+    <xacro:arg name="geometry_height" default="0.1" />
+    <xacro:arg name="geometry_radius" default="0.1" />
+    <xacro:arg name="geometry_length" default="0.1" />
+    <xacro:arg name="geometry_width" default="0.1" />
+    <xacro:arg name="geometry_mesh_filename" default="" />
+    <xacro:arg name="geometry_mesh_origin_xyz" default="0 0 0" />
+    <xacro:arg name="geometry_mesh_origin_rpy" default="0 0 0" />
+    <xacro:arg name="geometry_mesh_tcp_xyz" default="0 0 0" />
+    <xacro:arg name="geometry_mesh_tcp_rpy" default="0 0 0" />
+    <xacro:arg name="baud_checkset" default="true" />
+    <xacro:arg name="default_gripper_baud" default="2000000" />
+    <xacro:arg name="attach_to" default="$(arg prefix)base_link" />
+    <!-- <xacro:arg name="attach_xyz" default="0 0 0.5" /> -->
+    <xacro:arg name="attach_xyz" default="0 0 0.446" />
+    <xacro:arg name="attach_rpy" default="0 0 0" />
+    <xacro:arg name="mesh_suffix" default="stl" />
+    <xacro:arg name="kinematics_suffix" default="" />
     <xacro:include filename="$(find xarm_description)/urdf/xarm_device_macro.xacro" />
     <xacro:xarm_device prefix="$(arg prefix)" hw_ns="$(arg hw_ns)" limited="$(arg limited)"
-    effort_control="$(arg effort_control)" velocity_control="$(arg velocity_control)"
-    add_gripper="$(arg add_gripper)" add_vacuum_gripper="$(arg add_vacuum_gripper)" dof="$(arg dof)"
-    ros2_control_plugin="$(arg ros2_control_plugin)" robot_type="$(arg robot_type)"
-    load_gazebo_plugin="true" ros2_control_params="$(arg ros2_control_params)"
-    add_realsense_d435i="$(arg add_realsense_d435i)"
-    add_d435i_links="$(arg add_d435i_links)"
-    add_other_geometry="$(arg add_other_geometry)"
-    geometry_type="$(arg geometry_type)" geometry_mass="$(arg geometry_mass)"
-    geometry_height="$(arg geometry_height)" geometry_radius="$(arg geometry_radius)"
-    geometry_length="$(arg geometry_length)" geometry_width="$(arg geometry_width)"
-    geometry_mesh_filename="$(arg geometry_mesh_filename)"
-    geometry_mesh_origin_xyz="$(arg geometry_mesh_origin_xyz)" geometry_mesh_origin_rpy="$(arg geometry_mesh_origin_rpy)"
-    geometry_mesh_tcp_xyz="$(arg geometry_mesh_tcp_xyz)" geometry_mesh_tcp_rpy="$(arg geometry_mesh_tcp_rpy)"
-    robot_ip="$(arg robot_ip)" report_type="$(arg report_type)"
-    baud_checkset="$(arg baud_checkset)" default_gripper_baud="$(arg default_gripper_baud)"
-    model1300="$(arg model1300)" attach_to="$(arg attach_to)" attach_xyz="$(arg attach_xyz)" attach_rpy="$(arg attach_rpy)"
-    robot_sn="$(arg robot_sn)" use_gazebo_camera="$(arg use_gazebo_camera)" mesh_suffix="$(arg mesh_suffix)" kinematics_suffix="$(arg kinematics_suffix)" />
+        effort_control="$(arg effort_control)" velocity_control="$(arg velocity_control)"
+        add_gripper="$(arg add_gripper)" add_vacuum_gripper="$(arg add_vacuum_gripper)"
+        dof="$(arg dof)"
+        ros2_control_plugin="$(arg ros2_control_plugin)" robot_type="$(arg robot_type)"
+        load_gazebo_plugin="true" ros2_control_params="$(arg ros2_control_params)"
+        add_realsense_d435i="$(arg add_realsense_d435i)"
+        add_d435i_links="$(arg add_d435i_links)"
+        add_other_geometry="$(arg add_other_geometry)"
+        geometry_type="$(arg geometry_type)" geometry_mass="$(arg geometry_mass)"
+        geometry_height="$(arg geometry_height)" geometry_radius="$(arg geometry_radius)"
+        geometry_length="$(arg geometry_length)" geometry_width="$(arg geometry_width)"
+        geometry_mesh_filename="$(arg geometry_mesh_filename)"
+        geometry_mesh_origin_xyz="$(arg geometry_mesh_origin_xyz)"
+        geometry_mesh_origin_rpy="$(arg geometry_mesh_origin_rpy)"
+        geometry_mesh_tcp_xyz="$(arg geometry_mesh_tcp_xyz)"
+        geometry_mesh_tcp_rpy="$(arg geometry_mesh_tcp_rpy)"
+        robot_ip="$(arg robot_ip)" report_type="$(arg report_type)"
+        baud_checkset="$(arg baud_checkset)" default_gripper_baud="$(arg default_gripper_baud)"
+        model1300="$(arg model1300)" attach_to="$(arg attach_to)" attach_xyz="$(arg attach_xyz)"
+        attach_rpy="$(arg attach_rpy)"
+        robot_sn="$(arg robot_sn)" use_gazebo_camera="$(arg use_gazebo_camera)"
+        mesh_suffix="$(arg mesh_suffix)" kinematics_suffix="$(arg kinematics_suffix)" />
 </robot>
